File: kicad_9.0.1/STM32_USB_Buck_Converter/STM32_USB_Buck_Converter.kicad_sch (KiCad schematic)
At the start: 32 parts, among them Q1 AO3401A, SW1 SW_SPDT, U1 STM32F405RGT6, U2 MP2359DJ-LF-Z, Y1 16Mhz

Commit message: Finalizado
Parts:
- added D1: B5819W, Diode_SMD:D_SOD-123, symbol Device:D_Schottky_Small
- added D3: RED, LED_SMD:LED_0603_1608Metric, symbol Device:LED_Small
- added H1, H2, H3, H4: MountingHole_Pad, MountingHole:MountingHole_4.3mm_M4_Pad_Via, symbol Mechanical:MountingHole_Pad
- added J1: Screw_Terminal_01x02, TerminalBlock_Phoenix:TerminalBlock_Phoenix_PT-1,5-2-3.5-H_1x02_P3.50mm_Horizontal, symbol Connector:Screw_Terminal_01x02
- added J2: SWD, Connector_PinHeader_1.27mm:PinHeader_2x05_P1.27mm_Vertical_SMD, symbol Connector_Generic:Conn_02x05_Odd_Even
- added J3, J4: Conn_01x04, Connector_Molex:Molex_PicoBlade_53048-0410_1x04_P1.25mm_Horizontal, symbol Connector_Generic:Conn_01x04
- added J5: USB_B_Micro, USB_Connectors:USB_B_Micro, symbol Connector:USB_B_Micro
- added R10, R11: 2K2, Resistor_SMD:R_0402_1005Metric, symbol Device:R_Small
- added R3: 47K, Resistor_SMD:R_0603_1608Metric, symbol Device:R_Small
- added R4: 15K, Resistor_SMD:R_0603_1608Metric, symbol Device:R_Small
- added R5: 270, Resistor_SMD:R_0603_1608Metric, symbol Device:R_Small
- added R6: 1K, Resistor_SMD:R_0603_1608Metric, symbol Device:R_Small
- added U3: USBLC6-2SC6, Package_TO_SOT_SMD:SOT-23-6, symbol Power_Protection:USBLC6-2SC6
- C1: renamed from C13; footprint (none) -> Capacitor_SMD:C_1206_3216Metric; JLCPCB Part # (none) -> C13585
- C10: renamed from C8; footprint (none) -> Capacitor_SMD:C_0402_1005Metric; JLCPCB Part # (none) -> C1525
- C11: renamed from C9; footprint (none) -> Capacitor_SMD:C_0402_1005Metric; JLCPCB Part # (none) -> C52923
- C12: renamed from C10; footprint (none) -> Capacitor_SMD:C_0402_1005Metric; JLCPCB Part # (none) -> C1525
- C13: renamed from C1; footprint (none) -> Capacitor_SMD:C_0603_1608Metric; JLCPCB Part # (none) -> C15195
- C14: renamed from C3; footprint (none) -> Capacitor_SMD:C_0603_1608Metric; JLCPCB Part # (none) -> C15195
- C15: renamed from C11; footprint (none) -> Capacitor_SMD:C_0402_1005Metric; JLCPCB Part # (none) -> C1547
- C16: renamed from C12; footprint (none) -> Capacitor_SMD:C_0402_1005Metric; JLCPCB Part # (none) -> C1547
- C2: renamed from C15; footprint (none) -> Capacitor_SMD:C_1206_3216Metric; JLCPCB Part # (none) -> C13585
- C3: renamed from C16; footprint (none) -> Capacitor_SMD:C_1206_3216Metric; JLCPCB Part # (none) -> C13585
- C4: renamed from C14; footprint (none) -> Capacitor_SMD:C_0603_1608Metric; JLCPCB Part # (none) -> C57112
- C5: renamed from C2; footprint (none) -> Capacitor_SMD:C_0603_1608Metric; JLCPCB Part # (none) -> C19666
- C6: renamed from C4; footprint (none) -> Capacitor_SMD:C_0402_1005Metric; JLCPCB Part # (none) -> C1525
- C7: renamed from C5; footprint (none) -> Capacitor_SMD:C_0402_1005Metric; JLCPCB Part # (none) -> C1525
- C8: renamed from C6; footprint (none) -> Capacitor_SMD:C_0402_1005Metric; JLCPCB Part # (none) -> C1525
- C9: renamed from C7; footprint (none) -> Capacitor_SMD:C_0402_1005Metric; JLCPCB Part # (none) -> C1525
- D2: footprint (none) -> Diode_SMD:D_SOD-123; JLCPCB Part # (none) -> C8598
- D4: renamed from D1; footprint (none) -> LED_SMD:LED_0603_1608Metric; JLCPCB Part # (none) -> C72041; now not fitted
- F1: value 250mA -> 500mA; footprint (none) -> Fuse:Fuse_1206_3216Metric; JLCPCB Part # (none) -> C369159
- FB1: footprint (none) -> Inductor_SMD:L_0805_2012Metric; JLCPCB Part # (none) -> C1017
- L1: renamed from L2; footprint (none) -> Inductor_SMD:L_Sunlord_MWSA0518S; JLCPCB Part # (none) -> C139506
- L2: renamed from L1; footprint (none) -> Inductor_SMD:L_0402_1005Metric; JLCPCB Part # (none) -> C26443
- Q1: JLCPCB Part # (none) -> C15127
- R1: renamed from R4; footprint (none) -> Resistor_SMD:R_0603_1608Metric; JLCPCB Part # (none) -> C25803
- R2: renamed from R5; footprint (none) -> Resistor_SMD:R_0603_1608Metric; JLCPCB Part # (none) -> C23231
- R7: renamed from R2; footprint (none) -> Resistor_SMD:R_0402_1005Metric; JLCPCB Part # (none) -> C25744
- R8: renamed from R3; footprint (none) -> Resistor_SMD:R_0402_1005Metric; JLCPCB Part # (none) -> C25118
- R9: renamed from R1; footprint (none) -> Resistor_SMD:R_0603_1608Metric; JLCPCB Part # (none) -> C22843
- SW1: footprint (none) -> Button_Switch_SMD:SW_SPDT_PCM12
- U1: renamed from U2; footprint (none) -> Package_TO_SOT_SMD:SOT-23-6; JLCPCB Part # (none) -> C14259
- U2: renamed from U1; JLCPCB Part # (none) -> C15742
- Y1: footprint (none) -> Crystal:Crystal_SMD_3225-4Pin_3.2x2.5mm; JLCPCB Part # (none) -> C13738
Connections:
- net +12V: now also Q1.3 (D), J1.1 (Pin_1); no longer F1.1
- net +3.3V: now also D3.2 (A), J2.1 (Pin_1), J3.1 (Pin_1), J4.1 (Pin_1), R10.1, R11.1, R3.1
- net BUCK_FB: now also R3.2, R4.1
- net GND: now also H1.1, H2.1, H3.1, H4.1, J1.2 (Pin_2), J2.3 (Pin_3), J2.5 (Pin_5), J2.9 (Pin_9), J3.4 (Pin_4), J4.4 (Pin_4), J5.5 (GND), R5.2, R6.2, U3.2 (GND)
- net I2C1_SCL: now also J3.2 (Pin_2), R10.2
- net I2C1_SDA: now also J3.3 (Pin_3), R11.2
- net NRST: now also J2.10 (Pin_10)
- net SWCLK: now also J2.4 (Pin_4)
- net SWDIO: now also J2.2 (Pin_2)
- net SWO: now also J2.6 (Pin_6)
- net USART3_RX: now also J4.3 (Pin_3)
- net USART3_TX: now also J4.2 (Pin_2)
- net USB_D+: now also U3.4 (I/O2)
- net USB_D-: now also U3.6 (I/O1)
- net at FB1.1: now also F1.2; no longer Q1.2 (S)
- new net: R4.2, R5.1
- new net: D3.1 (K), R6.1
- new net: D1.1 (K), F1.1, Q1.2 (S)
- new net +5V: D1.2 (A), J5.1 (VBUS), U3.5 (VBUS)
- new net USB_CONN_D+: J5.3 (D+), U3.3 (I/O2)
- new net USB_CONN_D-: J5.2 (D-), U3.1 (I/O1)
- no-connect marks 39 -> 43
Other:
- note added: "Circuito de Alimentación"
- note added: "Conectores y USB"
- note added: "El inductor y el capacitor se calculan y seleccionan siguiendo la hoja de datos. Y es un POWER INDUCTOR al buscarlo en JLCPCB."
- note added: "El resistencia conectada al común, deberia valer 15,29K según la hoja de datos. En este caso, se ponen dos resistencias en serie para aproximarse a dicho valor."
- note added: "En este microcontrolador, no hace falta la resistencia de pull-up en USB_D+. Ver la nota de applicación 4879."
- note added: "La alimentación será de 12V a través del MOSFET aunque se conecte el cable USB porque el diodo schottky quedará polarizado en inversa. Si se quitan los 12V, se podrá alimentar la placa desde los +5V del USB."
- note added: "La distribución de pines del conector de debug es estándar."
- note added: "La protección ESD es necesaria porque el contector USB se va a enchufar y desenchufar varias veces por seres humanos que tienen cargar estática. La misma, se tiende a descargar a través del PCB. Colocar una protección, evita que la placa sufra daños."
- note added: "La protección contra polaridad inversa se hace con un MOSFET canal P. Se pierde menos potencia que con un diodo schottky (0,3V), porque tiene una RDS(ON) de 50m. La VGS máxima es de +/-12V, y es lo que limita la tensión de entrada. En caso de manejar más tensión, se debe utilizar un zener en el GATE."
- note added: "Lo comentado anteriormente de las resistencias de 22 también aplica para I2C y la USART/UART."
- note added: "NOTA: ENUMERAR LOS COMPONENTES MANUALMENTE"
- note added: "NOTA: LOS TAMAÑOS DE LOS COMPONENTES DE ESTA SECCIÓN SE ELIGEN GRANDES."
- note added: "NOTA: VER EN JLCPCB LOS TAMAÑOS DISPONIBLES PARA LOS COMPONENTES PASIVOS COLOCAR. USAR LOS BASIC, NO LOS EXTENDED."
- note added: "Perforaciones para sujetar el pcb mecánicamente."
- note added: "Resistencias de 2k2 de pull-up para 3.3V hasta 400Khz de SCL en I2C. Podrían ser de 4K7 para bajar el consumo. O de 10K si conectamos módulos externos que puedan tener las resistencias incluidas. Pueden ser 0805 por si hay que desoldar y cambiarlos. O 0402 si estamo seguros."
- note added: "Se recomienda colocar resistencias serie de valor 22 en los pines de los conectores para limitar las corrientes de cortocircuito en caso de una conexión errónea."
- note added: "Se recomienda colocar un capacitora a GND para evitar un reset parásito."
- note added: "Si no hay una carcasa metálica, dejar Shield sin conexión. No conectarlo a GND de forma direacta o mediante una resistencia y un capacitor. Sitios para buscar huellas: https://snapeda.com/"
- note added: "Siempre incluir leds que indiquen el estado de la alimentación"
- note removed: "El inductor y el capacitor se calculan y seleccionan siguiendo la hoja de datos."
- note removed: "La protección contra polaridad inversa se hace con un MOSFET canal P. Se pierde menos potencia que con un diodo schottky, porque tiene una RDS(ON) de 50m (baja). La VGS máxima es de +/-12V, y es lo que limita la tensión de entrada. En caso de manejar más tensión, se debe utilizar un zener en el GATE."
- moved on the sheet: C1, C11, C12, C2, C3, C4, D2, F1, FB1, L1, L2, Q1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
